Commit message: update project

File: install/assem1_description/share/assem1_description/urdf/ros2_control.xacro (robot description, xacro)
@@ -13,5 +13,5 @@
       </hardware>
     </xacro:unless>
-    <joint name="armlinl1">
+    <joint name="joint_1">
       <command_interface name="position">
         <param name="min">-3.1416</param>
@@ -21,5 +21,5 @@
       <state_interface name="velocity"/>
     </joint>
-    <joint name="armlinl2">
+    <joint name="joint_2">
       <command_interface name="position">
         <param name="min">-3.1416</param>

File: install/assem1_description/share/assem1_description/urdf/sensors.xacro (robot description, xacro)
@@ -17,5 +17,5 @@
             <origin xyz="0 0 0" rpy="0 0 0"/>
             <geometry>
-                <box size="0.1 0.1 0.05"/>
+                <box size="0.05 0.05 0.05"/>
             </geometry>
             <material name="red"/>
@@ -30,5 +30,5 @@
     <!-- ================= CAMERA JOINT ================= -->
     <joint name="camera_joint" type="fixed">
-        <origin xyz="-0.2 0.1 0.7" rpy="0 0 0"/>
+        <origin xyz="-0.2 0.1 0.7" rpy="0 1.57 0"/>
         <parent link="base_link"/>   <!-- مهم: مش panda_link0 -->
         <child link="camera_link"/>
