Commit message: back to zero

File: src/assem1_description/urdf/assem1.urdf.xacro (robot description, xacro)
@@ -1,9 +1,6 @@
 <?xml version="1.0"?>
-<robot name="assem1_robot" xmlns:xacro="http://www.ros.org/wiki/xacro">
-  <!-- مهم جدًا -->
-  <xacro:property name="pkg_name" value="assem1_description"/>
-  <!-- includes -->
+<robot name="assem1" xmlns:xacro="http://www.ros.org/wiki/xacro">
+  <xacro:arg name="is_ignition" default="true"/>
   <xacro:include filename="$(find assem1_description)/urdf/mobile_manipulator.xacro" />
-  <xacro:include filename="$(find assem1_description)/urdf/sensors.xacro" />
   <xacro:include filename="$(find assem1_description)/urdf/gazebo.xacro" />
   <xacro:include filename="$(find assem1_description)/urdf/ros2_control.xacro" />

File: src/assem1_description/urdf/gazebo.xacro (robot description, xacro)
@@ -1,32 +1,21 @@
 <?xml version="1.0"?>
-<robot xmlns:xacro="http://www.ros.org/wiki/xacro" name="assem1_robot">
-  <xacro:arg name="is_ignition" default="true"/>
+<robot xmlns:xacro="http://www.ros.org/wiki/xacro" name="Assem1">
   <gazebo>
-    <!-- ===== ROS 2 Humble ===== -->
     <xacro:if value="$(arg is_ignition)">
-      <plugin filename="ign_ros2_control-system"
-              name="ign_ros2_control::IgnitionROS2ControlPlugin">
-        <parameters>
-          $(find assem1_controller)/config/assem1_controllers.yaml
-        </parameters>
+      <plugin filename="ign_ros2_control-system" name="ign_ros2_control::IgnitionROS2ControlPlugin">
+        <parameters>$(find assem1_controller)/config/assem1_controllers.yaml</parameters>
       </plugin>
-      <plugin filename="ignition-gazebo-sensors-system"
-              name="ignition::gazebo::systems::Sensors">
+      <plugin filename="ignition-gazebo-sensors-system" name="ignition::gazebo::systems::Sensors">
         <render_engine>ogre2</render_engine>
       </plugin>
     </xacro:if>
-    <!-- ===== gz (Iron+) ===== -->
     <xacro:unless value="$(arg is_ignition)">
-      <plugin filename="gz_ros2_control-system"
-              name="gz_ros2_control::GazeboSimROS2ControlPlugin">
-        <parameters>
-          $(find assem1_controller)/config/assem1_controllers.yaml
-        </parameters>
+      <plugin filename="gz_ros2_control-system" name="gz_ros2_control::GazeboSimROS2ControlPlugin">
+        <parameters>$(find assem1_controller)/config/assem1_controllers.yaml</parameters>
       </plugin>
-      <plugin filename="gz-sim-sensors-system"
-              name="gz::sim::systems::Sensors">
+      <plugin filename="gz-sim-sensors-system" name="gz::sim::systems::Sensors">
         <render_engine>ogre2</render_engine>
       </plugin>
     </xacro:unless>
   </gazebo>
-</robot>
+  </robot>

File: src/assem1_description/urdf/mobile_manipulator.xacro (robot description, xacro)
@@ -1,65 +1,104 @@
-<?xml version="1.0"?>
-<robot name="assem1_robot" xmlns:xacro="http://www.ros.org/wiki/xacro">
-  <xacro:property name="pkg_name" value="assem1_description"/>
-  <material name="base_color"><color rgba="0.776 0.757 0.737 1"/></material>
-  <material name="arm_red"><color rgba="0.988 0.082 0 1"/></material>
-  <link name="world" />
-  <joint name="world_to_base_joint" type="fixed">
-    <parent link="world" /><child link="base_link" />
-    <origin xyz="0 0 0.304" rpy="0 0 0" />
+<?xml version="1.0" encoding="utf-8"?>
+<robot xmlns:xacro="http://www.ros.org/wiki/xacro">
+  <material name="silver"><color rgba="0.776 0.756 0.737 1" /></material>
+  <material name="dark_gray"><color rgba="0.3 0.3 0.3 1" /></material>
+  <material name="red_arm"><color rgba="0.988 0.082 0 1" /></material>
+  <link name="base_footprint"/>
+  <link name="support_left">
+    <inertial>
+      <mass value="5.0"/><inertia ixx="0.05" ixy="0" ixz="0" iyy="0.05" iyz="0" izz="0.05"/>
+    </inertial>
+    <visual>
+      <geometry><box size="0.6 0.3 0.15"/></geometry>
+      <material name="dark_gray"/>
+    </visual>
+    <collision>
+      <geometry><box size="0.6 0.3 0.15"/></geometry>
+    </collision>
+  </link>
+  <joint name="support_left_joint" type="fixed">
+    <parent link="base_footprint"/>
+    <child link="support_left"/>
+    <origin xyz="0.3 0.0 0.075" rpy="0 0 1.57"/>
+  </joint>
+  <link name="support_right">
+    <inertial>
+      <mass value="5.0"/><inertia ixx="0.05" ixy="0" ixz="0" iyy="0.05" iyz="0" izz="0.05"/>
+    </inertial>
+    <visual>
+      <geometry><box size="0.6 0.3 0.15"/></geometry>
+      <material name="dark_gray"/>
+    </visual>
+    <collision>
+      <geometry><box size="0.6 0.3 0.15"/></geometry>
+    </collision>
+  </link>
+  <joint name="support_right_joint" type="fixed">
+    <parent link="base_footprint"/>
+    <child link="support_right"/>
+    <origin xyz="-0.3 0.0 0.075" rpy="0 0 1.57"/>
   </joint>
   <link name="base_link">
     <inertial>
-      <origin xyz="0 0 0.2" rpy="0 0 0"/><mass value="36.0"/><inertia ixx="1.0" ixy="0" ixz="0" iyy="1.0" iyz="0" izz="1.0"/>
+      <origin xyz="-0.00155 0.0167 0.196" rpy="0 0 0" />
+      <mass value="36.7025" />
+      <inertia ixx="1.1928" ixy="-3.518E-06" ixz="1.993E-07" iyy="1.3331" iyz="0.00419" izz="1.3514" />
     </inertial>
     <visual>
-      <geometry><mesh filename="package://${pkg_name}/meshes/base_link.STL"/></geometry>
-      <material name="base_color"/>
+      <geometry><mesh filename="package://assem1_description/meshes/base_link.STL" /></geometry>
+      <material name="silver"/>
     </visual>
     <collision>
-      <geometry><mesh filename="package://${pkg_name}/meshes/base_link.STL"/></geometry>
+      <geometry><mesh filename="package://assem1_description/meshes/base_link.STL" /></geometry>
     </collision>
   </link>
-  <link name="armlink1">
+  <joint name="base_joint" type="fixed">
+    <parent link="base_footprint"/>
+    <child link="base_link"/>
+    <origin xyz="0 0 0.304" rpy="0 0 0"/>
+  </joint>
+  <link name="Armlink1">
     <inertial>
-      <origin xyz="0 0 0" rpy="0 0 0"/><mass value="1.0"/><inertia ixx="0.01" ixy="0" ixz="0" iyy="0.01" iyz="0" izz="0.01"/>
+      <origin xyz="0.00032 0.106 0.008" rpy="0 0 0" />
+      <mass value="0.3325" />
+      <inertia ixx="0.00125" ixy="0" ixz="0" iyy="6.2E-05" iyz="0" izz="0.00131" />
     </inertial>
     <visual>
-      <geometry><mesh filename="package://${pkg_name}/meshes/armlink1.STL"/></geometry>
-      <material name="arm_red"/>
+      <geometry><mesh filename="package://assem1_description/meshes/Armlink1.STL"/></geometry>
+      <material name="red_arm"/>
     </visual>
     <collision>
-      <geometry><mesh filename="package://${pkg_name}/meshes/armlink1.STL"/></geometry>
+      <geometry><mesh filename="package://assem1_description/meshes/Armlink1.STL"/></geometry>
     </collision>
   </link>
-  <joint name="joint_1" type="revolute">
-    <origin xyz="0 0.07 0.5" rpy="0 0 0"/>
-    <parent link="base_link"/><child link="armlink1"/>
+  <joint name="joint1" type="revolute">
+    <origin xyz="0 0.069976 0.4897" rpy="0 0 0" />
+    <parent link="base_link"/>
+    <child link="Armlink1"/>
     <axis xyz="0 0 1"/>
-    <limit lower="-1.2" upper="1.2" effort="100.0" velocity="3.0"/>
+    <limit lower="-0.785" upper="0.785" effort="10.0" velocity="1.0" />
   </joint>
   <link name="armlink2">
     <inertial>
-      <origin xyz="0 0 0" rpy="0 0 0"/><mass value="1.0"/><inertia ixx="0.01" ixy="0" ixz="0" iyy="0.01" iyz="0" izz="0.01"/>
+      <origin xyz="-0.00037 -0.094 -0.009" rpy="0 0 0" />
+      <mass value="0.3007" />
+      <inertia ixx="0.000749" ixy="0" ixz="0" iyy="7.2E-05" iyz="0" izz="0.000789" />
     </inertial>
     <visual>
-      <geometry><mesh filename="package://${pkg_name}/meshes/armlink2.STL"/></geometry>
-      <material name="arm_red"/>
+      <geometry><mesh filename="package://assem1_description/meshes/armlink2.STL"/></geometry>
+      <material name="red_arm"/>
     </visual>
     <collision>
-      <geometry><mesh filename="package://${pkg_name}/meshes/armlink2.STL"/></geometry>
+      <geometry><mesh filename="package://assem1_description/meshes/armlink2.STL"/></geometry>
     </collision>
   </link>
-  <joint name="joint_2" type="revolute">
-    <origin xyz="0 0.196 -0.02" rpy="0 0 0"/>
-    <parent link="armlink1"/><child link="armlink2"/>
+  <joint name="joint2" type="revolute">
+    <origin xyz="0.00077 0.19499 -0.0168" rpy="0 0 0" />
+    <parent link="Armlink1"/>
+    <child link="armlink2"/>
     <axis xyz="0 0 1"/>
-    <limit lower="-2.8" upper="2.8" effort="100.0" velocity="3.0"/>
+    <limit lower="-3.14" upper="3.14" effort="10.0" velocity="1.0" />
   </joint>
-  <link name="end_effector_point" />
-  <joint name="end_effector_joint" type="fixed">
-    <origin xyz="0 0.19 0" rpy="0 0 0"/>
-    <parent link="armlink2"/>
-    <child link="end_effector_point"/>
-  </joint>
+  <gazebo reference="support_left"><static>true</static></gazebo>
+  <gazebo reference="support_right"><static>true</static></gazebo>
 </robot>

File: src/assem1_description/urdf/ros2_control.xacro (robot description, xacro)
@@ -1,4 +1,4 @@
 <?xml version="1.0"?>
-<robot xmlns:xacro="http://www.ros.org/wiki/xacro" name="assem1_robot">
+<robot xmlns:xacro="http://www.ros.org/wiki/xacro" name="Assem1">
   <xacro:property name="PI" value="3.14159265359" />
   <ros2_control name="RobotSystem" type="system">
@@ -13,18 +13,22 @@
       </hardware>
     </xacro:unless>
-    <joint name="joint_1">
+    <joint name="joint1">
+      <command_interface name="position">
+        <param name="min">-0.785</param>
+        <param name="max">0.785</param>
+      </command_interface>
+      <state_interface name="position">
+        <param name="initial_value">0.0</param>
+      </state_interface>
+      <state_interface name="velocity"/>
+    </joint>
+    <joint name="joint2">
       <command_interface name="position">
         <param name="min">-3.1416</param>
         <param name="max">3.1416</param>
       </command_interface>
-      <state_interface name="position"/>
-      <state_interface name="velocity"/>
-    </joint>
-    <joint name="joint_2">
-      <command_interface name="position">
-        <param name="min">-3.1416</param>
-        <param name="max">3.1416</param>
-      </command_interface>
-      <state_interface name="position"/>
+      <state_interface name="position">
+        <param name="initial_value">0.0</param>
+      </state_interface>
       <state_interface name="velocity"/>
     </joint>

Commit message: Description&Control

File: src/assem1_description/urdf/assem1.urdf.xacro (robot description, xacro)
@@ -1,5 +1,4 @@
 <?xml version="1.0"?>
 <robot name="assem1" xmlns:xacro="http://www.ros.org/wiki/xacro">
-  <xacro:arg name="is_ignition" default="true"/>
   <xacro:include filename="$(find assem1_description)/urdf/mobile_manipulator.xacro" />
   <xacro:include filename="$(find assem1_description)/urdf/gazebo.xacro" />

File: src/assem1_description/urdf/gazebo.xacro (robot description, xacro)
@@ -1,4 +1,4 @@
 <?xml version="1.0"?>
-<robot xmlns:xacro="http://www.ros.org/wiki/xacro" name="Assem1">
+<robot xmlns:xacro="http://www.ros.org/wiki/xacro" name="assem1">
   <gazebo>
     <xacro:if value="$(arg is_ignition)">
@@ -19,3 +19,3 @@
     </xacro:unless>
   </gazebo>
-  </robot>
+</robot>

File: src/assem1_description/urdf/mobile_manipulator.xacro (robot description, xacro)
@@ -1,104 +1,80 @@
-<?xml version="1.0" encoding="utf-8"?>
+<?xml version="1.0"?>
 <robot xmlns:xacro="http://www.ros.org/wiki/xacro">
   <material name="silver"><color rgba="0.776 0.756 0.737 1" /></material>
   <material name="dark_gray"><color rgba="0.3 0.3 0.3 1" /></material>
   <material name="red_arm"><color rgba="0.988 0.082 0 1" /></material>
-  <link name="base_footprint"/>
-  <link name="support_left">
-    <inertial>
-      <mass value="5.0"/><inertia ixx="0.05" ixy="0" ixz="0" iyy="0.05" iyz="0" izz="0.05"/>
-    </inertial>
-    <visual>
-      <geometry><box size="0.6 0.3 0.15"/></geometry>
-      <material name="dark_gray"/>
-    </visual>
-    <collision>
-      <geometry><box size="0.6 0.3 0.15"/></geometry>
-    </collision>
-  </link>
-  <joint name="support_left_joint" type="fixed">
-    <parent link="base_footprint"/>
-    <child link="support_left"/>
-    <origin xyz="0.3 0.0 0.075" rpy="0 0 1.57"/>
-  </joint>
-  <link name="support_right">
-    <inertial>
-      <mass value="5.0"/><inertia ixx="0.05" ixy="0" ixz="0" iyy="0.05" iyz="0" izz="0.05"/>
-    </inertial>
-    <visual>
-      <geometry><box size="0.6 0.3 0.15"/></geometry>
-      <material name="dark_gray"/>
-    </visual>
-    <collision>
-      <geometry><box size="0.6 0.3 0.15"/></geometry>
-    </collision>
-  </link>
-  <joint name="support_right_joint" type="fixed">
-    <parent link="base_footprint"/>
-    <child link="support_right"/>
-    <origin xyz="-0.3 0.0 0.075" rpy="0 0 1.57"/>
+  <link name="world" />
+  <joint name="world_to_base_joint" type="fixed">
+    <parent link="world" />
+    <child link="base_link" />
+    <origin xyz="0 0 0" rpy="0 0 0" />
   </joint>
   <link name="base_link">
     <inertial>
-      <origin xyz="-0.00155 0.0167 0.196" rpy="0 0 0" />
-      <mass value="36.7025" />
-      <inertia ixx="1.1928" ixy="-3.518E-06" ixz="1.993E-07" iyy="1.3331" iyz="0.00419" izz="1.3514" />
+      <origin xyz="0 0 0" rpy="0 0 0"/>
+      <mass value="10"/>
+      <inertia ixx="0.1" ixy="0" ixz="0" iyy="0.1" iyz="0" izz="0.1"/>
     </inertial>
     <visual>
-      <geometry><mesh filename="package://assem1_description/meshes/base_link.STL" /></geometry>
+      <geometry>
+        <mesh filename="package://assem1_description/meshes/base_link.STL"/>
+      </geometry>
       <material name="silver"/>
     </visual>
     <collision>
-      <geometry><mesh filename="package://assem1_description/meshes/base_link.STL" /></geometry>
+      <geometry>
+        <mesh filename="package://assem1_description/meshes/base_link.STL"/>
+      </geometry>
     </collision>
   </link>
-  <joint name="base_joint" type="fixed">
-    <parent link="base_footprint"/>
-    <child link="base_link"/>
-    <origin xyz="0 0 0.304" rpy="0 0 0"/>
-  </joint>
-  <link name="Armlink1">
+  <link name="arm_link1">
     <inertial>
-      <origin xyz="0.00032 0.106 0.008" rpy="0 0 0" />
-      <mass value="0.3325" />
-      <inertia ixx="0.00125" ixy="0" ixz="0" iyy="6.2E-05" iyz="0" izz="0.00131" />
+      <origin xyz="0 0 0" rpy="0 0 0"/>
+      <mass value="1"/>
+      <inertia ixx="0.001" ixy="0" ixz="0" iyy="0.001" iyz="0" izz="0.001"/>
     </inertial>
     <visual>
-      <geometry><mesh filename="package://assem1_description/meshes/Armlink1.STL"/></geometry>
+      <geometry>
+        <mesh filename="package://assem1_description/meshes/Armlink1.STL"/>
+      </geometry>
       <material name="red_arm"/>
     </visual>
     <collision>
-      <geometry><mesh filename="package://assem1_description/meshes/Armlink1.STL"/></geometry>
+      <geometry>
+        <mesh filename="package://assem1_description/meshes/Armlink1.STL"/>
+      </geometry>
     </collision>
   </link>
-  <joint name="joint1" type="revolute">
-    <origin xyz="0 0.069976 0.4897" rpy="0 0 0" />
-    <parent link="base_link"/>
-    <child link="Armlink1"/>
-    <axis xyz="0 0 1"/>
-    <limit lower="-0.785" upper="0.785" effort="10.0" velocity="1.0" />
-  </joint>
-  <link name="armlink2">
+  <link name="arm_link2">
     <inertial>
-      <origin xyz="-0.00037 -0.094 -0.009" rpy="0 0 0" />
-      <mass value="0.3007" />
-      <inertia ixx="0.000749" ixy="0" ixz="0" iyy="7.2E-05" iyz="0" izz="0.000789" />
+      <origin xyz="0 0 0" rpy="0 0 0"/>
+      <mass value="1"/>
+      <inertia ixx="0.001" ixy="0" ixz="0" iyy="0.001" iyz="0" izz="0.001"/>
     </inertial>
     <visual>
-      <geometry><mesh filename="package://assem1_description/meshes/armlink2.STL"/></geometry>
+      <geometry>
+        <mesh filename="package://assem1_description/meshes/armlink2.STL"/>
+      </geometry>
       <material name="red_arm"/>
     </visual>
     <collision>
-      <geometry><mesh filename="package://assem1_description/meshes/armlink2.STL"/></geometry>
+      <geometry>
+        <mesh filename="package://assem1_description/meshes/armlink2.STL"/>
+      </geometry>
     </collision>
   </link>
-  <joint name="joint2" type="revolute">
-    <origin xyz="0.00077 0.19499 -0.0168" rpy="0 0 0" />
-    <parent link="Armlink1"/>
-    <child link="armlink2"/>
+  <joint name="joint_1" type="revolute">
+    <origin xyz="0 0.07 0.5" rpy="0 0 0"/>
+    <parent link="base_link"/>
+    <child link="arm_link1"/>
     <axis xyz="0 0 1"/>
-    <limit lower="-3.14" upper="3.14" effort="10.0" velocity="1.0" />
+    <limit lower="-0.785" upper="0.785" effort="100" velocity="3"/>
   </joint>
-  <gazebo reference="support_left"><static>true</static></gazebo>
-  <gazebo reference="support_right"><static>true</static></gazebo>
+  <joint name="joint_2" type="revolute">
+    <origin xyz="0 0.196 -0.02" rpy="0 0 0"/>
+    <parent link="arm_link1"/>
+    <child link="arm_link2"/>
+    <axis xyz="0 0 1"/>
+    <limit lower="-3.14" upper="3.14" effort="100" velocity="3"/>
+  </joint>
 </robot>

File: src/assem1_description/urdf/ros2_control.xacro (robot description, xacro)
@@ -1,4 +1,4 @@
 <?xml version="1.0"?>
-<robot xmlns:xacro="http://www.ros.org/wiki/xacro" name="Assem1">
+<robot xmlns:xacro="http://www.ros.org/wiki/xacro" name="assem1">
   <xacro:property name="PI" value="3.14159265359" />
   <ros2_control name="RobotSystem" type="system">
@@ -13,23 +13,17 @@
       </hardware>
     </xacro:unless>
-    <joint name="joint1">
+    <joint name="joint_1">
       <command_interface name="position">
         <param name="min">-0.785</param>
         <param name="max">0.785</param>
       </command_interface>
-      <state_interface name="position">
-        <param name="initial_value">0.0</param>
-      </state_interface>
-      <state_interface name="velocity"/>
+      <state_interface name="position"/>
     </joint>
-    <joint name="joint2">
+    <joint name="joint_2">
       <command_interface name="position">
-        <param name="min">-3.1416</param>
-        <param name="max">3.1416</param>
+        <param name="min">-3.14</param>
+        <param name="max">3.14</param>
       </command_interface>
-      <state_interface name="position">
-        <param name="initial_value">0.0</param>
-      </state_interface>
-      <state_interface name="velocity"/>
+      <state_interface name="position"/>
     </joint>
   </ros2_control>

File: src/assem1_description/urdf/sensors.xacro (robot description, xacro)
@@ -1,4 +1,4 @@
 <?xml version="1.0" ?>
-<robot name="assem1_robot" xmlns:xacro="http://www.ros.org/wiki/xacro">
+<robot name="assem1" xmlns:xacro="http://www.ros.org/wiki/xacro">
     <!-- ================= PROPERTIES ================= -->
     <xacro:property name="PI" value="3.14159265359"/>

Commit message: des,con,vision

File: src/assem1_description/urdf/assem1.urdf.xacro (robot description, xacro)
@@ -4,3 +4,4 @@
   <xacro:include filename="$(find assem1_description)/urdf/gazebo.xacro" />
   <xacro:include filename="$(find assem1_description)/urdf/ros2_control.xacro" />
+  <xacro:include filename="$(find assem1_description)/urdf/sensors.xacro" />
 </robot>

File: src/assem1_description/urdf/mobile_manipulator.xacro (robot description, xacro)
@@ -1,13 +1,8 @@
 <?xml version="1.0"?>
-<robot xmlns:xacro="http://www.ros.org/wiki/xacro">
+<robot name="assem1" xmlns:xacro="http://www.ros.org/wiki/xacro">
   <material name="silver"><color rgba="0.776 0.756 0.737 1" /></material>
   <material name="dark_gray"><color rgba="0.3 0.3 0.3 1" /></material>
   <material name="red_arm"><color rgba="0.988 0.082 0 1" /></material>
   <link name="world" />
-  <joint name="world_to_base_joint" type="fixed">
-    <parent link="world" />
-    <child link="base_link" />
-    <origin xyz="0 0 0" rpy="0 0 0" />
-  </joint>
   <link name="base_link">
     <inertial>
@@ -28,4 +23,9 @@
     </collision>
   </link>
+  <joint name="virtual_joint" type="fixed">
+      <parent link="world"/>
+      <child link="base_link"/>
+      <origin xyz="0 0 0" rpy="0 0 0"/>
+  </joint>
   <link name="arm_link1">
     <inertial>
