Commit message: befor  moveit

File: src/assem1_description/urdf/mobile_manipulator.xacro (robot description, xacro)
@@ -2,116 +2,58 @@
 <robot name="assem1_robot" xmlns:xacro="http://www.ros.org/wiki/xacro">
   <xacro:property name="pkg_name" value="assem1_description"/>
-  <xacro:property name="PI" value="3.1415926535897931"/>
-  <!-- ================= MATERIALS ================= -->
-  <material name="base_color">
-    <color rgba="0.776 0.757 0.737 1"/>
-  </material>
-  <material name="arm_red">
-    <color rgba="0.988 0.082 0 1"/>
-  </material>
-  <!-- ================ worlds   ==================== -->
+  <material name="base_color"><color rgba="0.776 0.757 0.737 1"/></material>
+  <material name="arm_red"><color rgba="0.988 0.082 0 1"/></material>
   <link name="world" />
   <joint name="world_to_base_joint" type="fixed">
-    <parent link="world" />
-    <child link="base_link" />
+    <parent link="world" /><child link="base_link" />
     <origin xyz="0 0 0" rpy="0 0 0" />
   </joint>
-  <!-- ================= BASE LINK ================= -->
   <link name="base_link">
     <inertial>
-      <origin xyz="0 0 0" rpy="0 0 0"/>
-      <mass value="10"/>
-      <inertia ixx="0.1" ixy="0" ixz="0" iyy="0.1" iyz="0" izz="0.1"/>
+      <origin xyz="0 0 0.2" rpy="0 0 0"/><mass value="36.0"/><inertia ixx="1.0" ixy="0" ixz="0" iyy="1.0" iyz="0" izz="1.0"/>
     </inertial>
     <visual>
-      <geometry>
-        <mesh filename="package://${pkg_name}/meshes/base_link.STL"/>
-      </geometry>
+      <geometry><mesh filename="package://${pkg_name}/meshes/base_link.STL"/></geometry>
       <material name="base_color"/>
     </visual>
     <collision>
-      <geometry>
-        <mesh filename="package://${pkg_name}/meshes/base_link.STL"/>
-      </geometry>
+      <geometry><mesh filename="package://${pkg_name}/meshes/base_link.STL"/></geometry>
     </collision>
   </link>
-  <!-- ================= ARM LINK 1 ================= -->
-  <link name="arm_link1">
+  <link name="armlink1">
     <inertial>
-      <origin xyz="0 0 0" rpy="0 0 0"/>
-      <mass value="1"/>
-      <inertia ixx="0.001" ixy="0" ixz="0" iyy="0.001" iyz="0" izz="0.001"/>
+      <origin xyz="0 0 0" rpy="0 0 0"/><mass value="1.0"/><inertia ixx="0.01" ixy="0" ixz="0" iyy="0.01" iyz="0" izz="0.01"/>
     </inertial>
     <visual>
-      <geometry>
-        <mesh filename="package://${pkg_name}/meshes/armlink1.STL"/>
-      </geometry>
+      <geometry><mesh filename="package://${pkg_name}/meshes/armlink1.STL"/></geometry>
       <material name="arm_red"/>
     </visual>
     <collision>
-      <geometry>
-        <mesh filename="package://${pkg_name}/meshes/armlink1.STL"/>
-      </geometry>
+      <geometry><mesh filename="package://${pkg_name}/meshes/armlink1.STL"/></geometry>
     </collision>
   </link>
-  <!-- ================= ARM LINK 2 ================= -->
-  <link name="arm_link2">
+  <joint name="joint_1" type="revolute">
+    <origin xyz="0 0.07 0.5" rpy="0 0 0"/>
+    <parent link="base_link"/><child link="armlink1"/>
+    <axis xyz="0 0 1"/>
+    <limit lower="-1.2" upper="1.2" effort="100" velocity="3"/>
+  </joint>
+  <link name="armlink2">
     <inertial>
-      <origin xyz="0 0 0" rpy="0 0 0"/>
-      <mass value="1"/>
-      <inertia ixx="0.001" ixy="0" ixz="0" iyy="0.001" iyz="0" izz="0.001"/>
+      <origin xyz="0 0 0" rpy="0 0 0"/><mass value="1.0"/><inertia ixx="0.01" ixy="0" ixz="0" iyy="0.01" iyz="0" izz="0.01"/>
     </inertial>
     <visual>
-      <geometry>
-        <mesh filename="package://${pkg_name}/meshes/armlink2.STL"/>
-      </geometry>
+      <geometry><mesh filename="package://${pkg_name}/meshes/armlink2.STL"/></geometry>
       <material name="arm_red"/>
     </visual>
     <collision>
-      <geometry>
-        <mesh filename="package://${pkg_name}/meshes/armlink2.STL"/>
-      </geometry>
+      <geometry><mesh filename="package://${pkg_name}/meshes/armlink2.STL"/></geometry>
     </collision>
   </link>
-  <!-- ================= end effector ============ -->
-  <link name="tool_link">
-    <inertial>
-      <mass value="0.1"/>
-      <origin xyz="0 0 0" rpy="0 0 0"/>
-      <inertia ixx="0.001" ixy="0" ixz="0" iyy="0.001" iyz="0" izz="0.001"/>
-    </inertial>
-    <visual>
-      <geometry>
-        <cylinder radius="0.028" length="0.0097" />
-      </geometry>
-      <material name="base_color"/>
-    </visual>
-    <collision>
-      <geometry>
-        <cylinder radius="0.028" length="0.0097" />
-      </geometry>
-    </collision>
-  </link>
-  <!-- ================= JOINT 1 ================= -->
-  <joint name="joint_1" type="revolute">
-    <origin xyz="0 0.07 0.5" rpy="0 0 0"/>
-    <parent link="base_link"/>
-    <child link="arm_link1"/>
-    <axis xyz="0 0 1"/>
-    <limit lower="-${PI/2}" upper="${PI/2}" effort="100" velocity="3"/>
-  </joint>
-  <!-- ================= JOINT 2 ================= -->
   <joint name="joint_2" type="revolute">
     <origin xyz="0 0.196 -0.02" rpy="0 0 0"/>
-    <parent link="arm_link1"/>
-    <child link="arm_link2"/>
+    <parent link="armlink1"/><child link="armlink2"/>
     <axis xyz="0 0 1"/>
-    <limit lower="-${PI}" upper="${PI}" effort="100" velocity="3"/>
-  </joint>
-  <!-- ================= JOINT 3 ================= -->
-  <joint name="tool_joint" type="fixed">
-    <origin xyz="0 -0.165 -0.107" rpy="0 0 0"/>
-    <parent link="arm_link2"/>
-    <child link="tool_link"/>
+    <limit lower="-2.8" upper="2.8" effort="100" velocity="3"/>
   </joint>
 </robot>

Commit message: edit

File: src/assem1_description/urdf/mobile_manipulator.xacro (robot description, xacro)
@@ -7,5 +7,5 @@
   <joint name="world_to_base_joint" type="fixed">
     <parent link="world" /><child link="base_link" />
-    <origin xyz="0 0 0" rpy="0 0 0" />
+    <origin xyz="0 0 0.304" rpy="0 0 0" />
   </joint>
   <link name="base_link">
@@ -37,5 +37,5 @@
     <parent link="base_link"/><child link="armlink1"/>
     <axis xyz="0 0 1"/>
-    <limit lower="-1.2" upper="1.2" effort="100" velocity="3"/>
+    <limit lower="-1.2" upper="1.2" effort="100.0" velocity="3.0"/>
   </joint>
   <link name="armlink2">
@@ -55,5 +55,24 @@
     <parent link="armlink1"/><child link="armlink2"/>
     <axis xyz="0 0 1"/>
-    <limit lower="-2.8" upper="2.8" effort="100" velocity="3"/>
+    <limit lower="-2.8" upper="2.8" effort="100.0" velocity="3.0"/>
   </joint>
+  <link name="end_effector_point" />
+  <joint name="end_effector_joint" type="fixed">
+    <origin xyz="0 0.19 0" rpy="0 0 0"/>
+    <parent link="armlink2"/>
+    <child link="end_effector_point"/>
+  </joint>
+  <ros2_control name="FakeSystem" type="system">
+    <hardware>
+      <plugin>mock_components/GenericSystem</plugin>
+    </hardware>
+    <joint name="joint_1">
+      <command_interface name="position"/>
+      <state_interface name="position"/>
+      <state_interface name="velocity"/> </joint>
+    <joint name="joint_2">
+      <command_interface name="position"/>
+      <state_interface name="position"/>
+      <state_interface name="velocity"/> </joint>
+  </ros2_control>
 </robot>

Commit message: edit

File: src/assem1_description/urdf/mobile_manipulator.xacro (robot description, xacro)
@@ -63,16 +63,3 @@
     <child link="end_effector_point"/>
   </joint>
-  <ros2_control name="FakeSystem" type="system">
-    <hardware>
-      <plugin>mock_components/GenericSystem</plugin>
-    </hardware>
-    <joint name="joint_1">
-      <command_interface name="position"/>
-      <state_interface name="position"/>
-      <state_interface name="velocity"/> </joint>
-    <joint name="joint_2">
-      <command_interface name="position"/>
-      <state_interface name="position"/>
-      <state_interface name="velocity"/> </joint>
-  </ros2_control>
 </robot>

Commit message: collosion edit

File: src/assem1_description/urdf/mobile_manipulator.xacro (robot description, xacro)
@@ -6,9 +6,4 @@
   <link name="world" />
   <link name="base_link">
-    <inertial>
-      <origin xyz="0 0 0" rpy="0 0 0"/>
-      <mass value="10"/>
-      <inertia ixx="0.1" ixy="0" ixz="0" iyy="0.1" iyz="0" izz="0.1"/>
-    </inertial>
     <visual>
       <geometry>
@@ -18,8 +13,24 @@
     </visual>
     <collision>
+      <origin
+        xyz="0 0 0" rpy="0 0 0" />
       <geometry>
         <mesh filename="package://assem1_description/meshes/base_link.STL"/>
       </geometry>
     </collision>
+    <inertial>
+      <origin
+        xyz="-0.00155506458890642 -0.0167350728595071 0.196068139571374"
+        rpy="0 0 0" />
+      <mass
+        value="36.7025357857225" />
+      <inertia
+        ixx="1.19283308759496"
+        ixy="-3.51896300637401E-06"
+        ixz="1.99354682337673E-07"
+        iyy="1.33312260434488"
+        iyz="0.00419911892440131"
+        izz="1.35147505804967" />
+    </inertial>
   </link>
   <joint name="virtual_joint" type="fixed">
@@ -29,9 +40,4 @@
   </joint>
   <link name="arm_link1">
-    <inertial>
-      <origin xyz="0 0 0" rpy="0 0 0"/>
-      <mass value="1"/>
-      <inertia ixx="0.001" ixy="0" ixz="0" iyy="0.001" iyz="0" izz="0.001"/>
-    </inertial>
     <visual>
       <geometry>
@@ -41,15 +47,34 @@
     </visual>
     <collision>
+      <origin
+        xyz="0 0 0" rpy="0 0 0" />
       <geometry>
         <mesh filename="package://assem1_description/meshes/Armlink1.STL"/>
       </geometry>
     </collision>
+    <inertial>
+      <origin
+        xyz="0.0003200901517868 0.10625947606417 0.00859769829677659"
+        rpy="0 0 0" />
+      <mass
+        value="0.332522666985014" />
+      <inertia
+        ixx="0.00125293093936372"
+        ixy="-4.70356148528572E-06"
+        ixz="3.39571390138256E-10"
+        iyy="6.28321938668438E-05"
+        iyz="7.22390011604219E-08"
+        izz="0.00131069685758587" />
+    </inertial>
   </link>
+  <joint name="joint_1" type="revolute">
+    <origin
+      xyz="0 0.069976 0.4897" rpy="0 0 0" />
+    <parent link="base_link"/>
+    <child link="arm_link1"/>
+    <axis xyz="0 0 1"/>
+    <limit lower="-0.785" upper="0.785" effort="100" velocity="3"/>
+  </joint>
   <link name="arm_link2">
-    <inertial>
-      <origin xyz="0 0 0" rpy="0 0 0"/>
-      <mass value="1"/>
-      <inertia ixx="0.001" ixy="0" ixz="0" iyy="0.001" iyz="0" izz="0.001"/>
-    </inertial>
     <visual>
       <geometry>
@@ -59,18 +84,27 @@
     </visual>
     <collision>
+      <origin
+        xyz="0 0 0" rpy="0 0 0" />
       <geometry>
         <mesh filename="package://assem1_description/meshes/armlink2.STL"/>
       </geometry>
     </collision>
+    <inertial>
+      <origin
+        xyz="-0.000378523464681146 -0.0941307105712545 -0.00947503989193477"
+        rpy="0 0 0" />
+      <mass
+        value="0.300704203880306" />
+      <inertia
+        ixx="0.000749795032834774"
+        ixy="-2.68858863020437E-06"
+        ixz="3.21601810886238E-08"
+        iyy="7.27567345311832E-05"
+        iyz="-4.00235469561631E-08"
+        izz="0.000789914137832894" />
+    </inertial>
   </link>
-  <joint name="joint_1" type="revolute">
-    <origin xyz="0 0.07 0.5" rpy="0 0 0"/>
-    <parent link="base_link"/>
-    <child link="arm_link1"/>
-    <axis xyz="0 0 1"/>
-    <limit lower="-0.785" upper="0.785" effort="100" velocity="3"/>
-  </joint>
   <joint name="joint_2" type="revolute">
-    <origin xyz="0 0.196 -0.02" rpy="0 0 0"/>
+    <origin xyz="0.00077145 0.194994 -0.0168" rpy="0 0 0"/>
     <parent link="arm_link1"/>
     <child link="arm_link2"/>

File: src/assem1_description/urdf/sensors.xacro (robot description, xacro)
@@ -22,7 +22,7 @@
         </visual>
         <collision>
-            <origin xyz="0.2 0.1 1" rpy="0 0 0"/>
+            <origin xyz="0 0 0" rpy="0 0 0"/>
             <geometry>
-                <box size="0.1 0.1 0.05"/>
+                <box size="0.05 0.05 0.05"/>
             </geometry>
         </collision>
