Commit message: all pkg

File: src/assem_description/urdf/sensors.xacro (robot description, xacro)
@@ -17,5 +17,5 @@
             <origin xyz="0 0 0" rpy="0 0 0"/>
             <geometry>
-                <box size="0.05 0.05 0.05"/>
+               <box size="0.05 0.05 0.05"/>
             </geometry>
             <material name="red"/>
@@ -31,5 +31,5 @@
     <joint name="camera_joint" type="fixed">
         <origin xyz="-0.2 0.1 0.7" rpy="0 1.57 0"/>
-        <parent link="base_link"/>   <!-- مهم: مش panda_link0 -->
+        <parent link="base_link"/>
         <child link="camera_link"/>
     </joint>
