Commit message: moveit done

File: src/assem_description/urdf/mobile_manipulator.xacro (robot description, xacro)
@@ -74,5 +74,5 @@
     <child link="arm_link1"/>
     <axis xyz="0 0 1"/>
-    <limit lower="-0.785" upper="0.785" effort="100" velocity="3"/>
+    <limit lower="-0.785" upper="0.785" effort="100.0" velocity="3.0"/>
   </joint>
   <link name="arm_link2">
@@ -110,5 +110,5 @@
     <child link="arm_link2"/>
     <axis xyz="0 0 1"/>
-    <limit lower="-3.14" upper="3.14" effort="100" velocity="3"/>
+    <limit lower="-3.14" upper="3.14" effort="100.0" velocity="3.0"/>
   </joint>
 </robot>

Commit message: edit collision

File: src/assem_description/urdf/mobile_manipulator.xacro (robot description, xacro)
@@ -16,5 +16,5 @@
         xyz="0 0 0" rpy="0 0 0" />
       <geometry>
-        <mesh filename="package://assem_description/meshes/base_link.STL"/>
+        <mesh filename="package://assem_description/meshes/collision/base_link.obj"/>
       </geometry>
     </collision>
@@ -50,5 +50,5 @@
         xyz="0 0 0" rpy="0 0 0" />
       <geometry>
-        <mesh filename="package://assem_description/meshes/Armlink1.STL"/>
+        <mesh filename="package://assem_description/meshes/collision/Armlink1.obj"/>
       </geometry>
     </collision>
@@ -87,5 +87,5 @@
         xyz="0 0 0" rpy="0 0 0" />
       <geometry>
-        <mesh filename="package://assem_description/meshes/armlink2.STL"/>
+        <mesh filename="package://assem_description/meshes/collision/armlink2.obj"/>
       </geometry>
     </collision>
@@ -112,3 +112,39 @@
     <limit lower="-3.14" upper="3.14" effort="100.0" velocity="3.0"/>
   </joint>
+  <!-- <link name="suction_cup">
+    <visual>
+      <geometry>
+        <cylinder radius="0.028" length="0.0097" />
+      </geometry>
+      <material name="dark_gray"/>
+    </visual>
+    <collision>
+      <origin
+        xyz="0 0 0" rpy="0 0 0" />
+      <geometry>
+        <cylinder radius="0.028" length="0.0097" />
+      </geometry>
+    </collision>
+    <inertial>
+      <origin
+        xyz="-0.0 0.0 0.0"
+        rpy="0 0 0" />
+      <mass
+        value="0.1" />
+      <inertia
+        ixx="0.001"
+        ixy="0.0"
+        ixz="0.0"
+        iyy="0.001"
+        iyz="0.0"
+        izz="0.001" />
+    </inertial>
+  </link>
+  <joint name="joint_3" type="fixed">
+    <origin xyz="0.0 -0.165 -0.107" rpy="0 0 0"/>
+    <parent link="arm_link2"/>
+    <child link="suction_cup"/>
+    <axis xyz="0 0 1"/>
+    <limit lower="-3.14" upper="3.14" effort="100.0" velocity="3.0"/>
+  </joint>-->
 </robot>

Commit message: all structure

File: src/assem_description/urdf/mobile_manipulator.xacro (robot description, xacro)
@@ -16,5 +16,5 @@
         xyz="0 0 0" rpy="0 0 0" />
       <geometry>
-        <mesh filename="package://assem_description/meshes/collision/base_link.obj"/>
+        <mesh filename="package://assem_description/meshes/base_link.STL"/>
       </geometry>
     </collision>
@@ -50,5 +50,5 @@
         xyz="0 0 0" rpy="0 0 0" />
       <geometry>
-        <mesh filename="package://assem_description/meshes/collision/Armlink1.obj"/>
+        <mesh filename="package://assem_description/meshes/Armlink1.STL"/>
       </geometry>
     </collision>
@@ -87,5 +87,5 @@
         xyz="0 0 0" rpy="0 0 0" />
       <geometry>
-        <mesh filename="package://assem_description/meshes/collision/armlink2.obj"/>
+        <mesh filename="package://assem_description/meshes/armlink2.STL"/>
       </geometry>
     </collision>
