Commit message: go to color

File: src/assem_description/urdf/gazebo.xacro (robot description, xacro)
@@ -1,7 +1,6 @@
 <?xml version="1.0"?>
 <robot xmlns:xacro="http://www.ros.org/wiki/xacro" name="assem">
-  <!-- ROS 2 Control -->
   <gazebo>
-    <!-- ROS 2 Humble (Ignition Gazebo) -->
+    <!-- 1. حالة ROS 2 Humble (Ignition Gazebo) -->
     <xacro:if value="$(arg is_ignition)">
       <plugin filename="ign_ros2_control-system" name="ign_ros2_control::IgnitionROS2ControlPlugin">
@@ -11,6 +10,12 @@
         <render_engine>ogre2</render_engine>
       </plugin>
+      <!-- تم تصحيح filename وإزالة f الزائدة -->
+    <!--   <plugin filename="ignition-gazebo-vacuum-gripper-system" name="ignition::gazebo::systems::VacuumGripper">
+        <topic>/assem/switch_suction</topic>
+        <link_name>suction_cup</link_name>
+        <max_distance>0.02</max_distance>
+      </plugin>-->
     </xacro:if>
-    <!-- ROS 2 Jazzy or Iron (Gazebo Sim) -->
+    <!-- 2. حالة ROS 2 Jazzy (Gazebo Sim - Harmonic) -->
     <xacro:unless value="$(arg is_ignition)">
       <plugin filename="gz_ros2_control-system" name="gz_ros2_control::GazeboSimROS2ControlPlugin">
@@ -20,6 +25,11 @@
         <render_engine>ogre2</render_engine>
       </plugin>
-      <plugin filename="gz-sim-scene-broadcaster-system" name="gz::sim::systems::SceneBroadcaster">
+      <!-- تم تحديث اسم المكتبة ليتوافق مع Gazebo Harmonic في Jazzy -->
+      <plugin filename="gz-sim-vacuum-gripper-system" name="gz::sim::systems::VacuumGripper">
+        <topic>/assem/switch_suction</topic>
+        <link_name>suction_cup</link_name>
+        <max_distance>0.05</max_distance>
       </plugin>
+      <plugin filename="gz-sim-scene-broadcaster-system" name="gz::sim::systems::SceneBroadcaster"/>
     </xacro:unless>
   </gazebo>

File: src/assem_description/urdf/mobile_manipulator.xacro (robot description, xacro)
@@ -112,5 +112,5 @@
     <limit lower="-3.14" upper="3.14" effort="100.0" velocity="3.0"/>
   </joint>
-  <!-- <link name="suction_cup">
+  <link name="suction_cup">
     <visual>
       <geometry>
@@ -147,4 +147,4 @@
     <axis xyz="0 0 1"/>
     <limit lower="-3.14" upper="3.14" effort="100.0" velocity="3.0"/>
-  </joint>-->
+  </joint>
 </robot>

File: src/assem_description/urdf/sensors.xacro (robot description, xacro)
@@ -1,64 +1,53 @@
 <?xml version="1.0" ?>
 <robot name="assem" xmlns:xacro="http://www.ros.org/wiki/xacro">
-    <!-- ================= PROPERTIES ================= -->
-    <xacro:property name="PI" value="3.14159265359"/>
-    <!-- ================= MATERIAL ================= -->
-    <material name="red">
-        <color rgba="1 0 0 1"/>
-    </material>
-    <!-- ================= CAMERA LINK ================= -->
     <link name="camera_link">
         <inertial>
-            <origin xyz="0 0 0" rpy="0 0 0"/>
+            <origin xyz="0 0 0" rpy="0.0 0.0 0.0"/>
             <mass value="0.1"/>
-            <inertia ixx="0.01" ixy="0" ixz="0" iyy="0.01" iyz="0" izz="0.01"/>
+            <inertia ixx="0.1" ixy="0.0" ixz="0.0" iyy="0.1" iyz="0.0" izz="0.1"/>
         </inertial>
         <visual>
-            <origin xyz="0 0 0" rpy="0 0 0"/>
+            <origin xyz="0 0 0" rpy="0.0 0.0 0.0"/>
             <geometry>
-               <box size="0.05 0.05 0.05"/>
+                <box size="0.1 0.1 0.05"/>
             </geometry>
             <material name="red"/>
         </visual>
         <collision>
-            <origin xyz="0 0 0" rpy="0 0 0"/>
+            <origin xyz="0 0 0" rpy="0.0 0.0 0.0"/>
             <geometry>
-                <box size="0.05 0.05 0.05"/>
+                <box size="0.1 0.1 0.05"/>
             </geometry>
         </collision>
     </link>
-    <!-- ================= CAMERA JOINT ================= -->
     <joint name="camera_joint" type="fixed">
-        <origin xyz="-0.2 0.1 0.7" rpy="0 1.57 0"/>
+        <origin xyz="-0.2 0.1 0.7" rpy="0.0 0.0 0.0"/>
         <parent link="base_link"/>
         <child link="camera_link"/>
     </joint>
-    <!-- ================= OPTICAL FRAME ================= -->
-    <link name="camera_link_optical"/>
+    <link name="camera_link_optical" />
     <joint name="camera_optical_joint" type="fixed">
         <parent link="camera_link"/>
         <child link="camera_link_optical"/>
-        <origin xyz="0 0 0" rpy="${-PI/2} 0 ${-PI/2}"/>
+        <origin xyz="0 0 0" rpy="${-pi/2} 0 ${-pi/2}"/>
     </joint>
-    <!-- ================= GAZEBO CAMERA ================= -->
     <gazebo reference="camera_link">
         <sensor name="camera" type="camera">
-            <pose>0 0 0 0 0 0</pose>
+            <pose>0 0 0 0 1.57 0</pose>
             <visualize>true</visualize>
-            <update_rate>30.0</update_rate>
-            <always_on>true</always_on>
-            <topic>/camera/image_raw</topic>
+            <update_rate>10.0</update_rate>
+            <topic>camera/image_raw</topic>
             <gz_frame_id>camera_link_optical</gz_frame_id>
-            <camera name="rgb_camera">
-                <camera_info_topic>/camera/camera_info</camera_info_topic>
-                <horizontal_fov>1.047</horizontal_fov>
+            <camera name="intel_realsense_r200">
+                <camera_info_topic>camera/camera_info</camera_info_topic>
+                <horizontal_fov>1.0</horizontal_fov>
                 <image>
                     <width>640</width>
-                    <height>480</height>
+                    <height>320</height>
                     <format>R8G8B8</format>
                 </image>
                 <clip>
                     <near>0.05</near>
-                    <far>10.0</far>
+                    <far>8.0</far>
                 </clip>
             </camera>
